File: LM5146Buck/LM5146Buck.kicad_sch (KiCad schematic)
At the start: 0 parts

Commit message: Update LM5146Buck.kicad_sch
Parts:
- added U?: LM5146RGYR, 0_LM5146:IC_LM5146RGYR, symbol 0_LM5146RGYR:LM5146RGYR
Connections:
- new net: U?.16 (NC), U?.9 (NC)
- new net EP: U?.15 (EP), U?.21 (EP)

Commit message: Update LM5146Buck.kicad_sch
Parts:
- added C1: 100n, Capacitor_SMD:C_0603_1608Metric, symbol Device:C
- added Q? (x2): (no value), Package_TO_SOT_SMD:TDSON-8-1, symbol Transistor_FET:BSC123N10LSG
- added R1: 511, Resistor_SMD:R_0603_1608Metric, symbol Device:R
- added R2: 10k2, Resistor_SMD:R_0603_1608Metric, symbol Device:R
- added R3: R, Resistor_SMD:R_0603_1608Metric, symbol Device:R
- U?: CREATOR DIZAR -> (none); Check_prices https://www.snapeda.com/parts/LM5146RGYR/Texas+Instruments/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 -> (none); DUPLICATE LM5146RGYR.A-,-LM5146RGYRG4-,-LM5146RGYRG4.A -> (none); DigiKey_Part_Number 296-LM5146RGYRCT-ND -> (none); MANUFACTURER Texas Instruments -> (none); MAXIMUM_PACKAGE_HEIGHT 1.0mm -> (none); MF Texas Instruments -> (none); MP LM5146RGYR -> (none); PARTREV A -> (none); Package VFQFN-20 Texas Instruments -> (none); STANDARD Manufacturer Recommendations -> (none); SnapEDA_Link https://www.snapeda.com/parts/LM5146RGYR/Texas+Instruments/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 -> (none)
Connections:
- net GND: now reaches U?.12 (PGND)
- net GND: now also U?.6 (AGND)
- net LO_MOSFET_G: now reaches U?.13 (LO)
- net LO_MOSFET_G: now also Q?.4 (G)
- net HO_MOSFET_G: now reaches U?.18 (HO)
- net HO_MOSFET_G: now also Q?.4 (G)
- new net: Q?.1 (S), Q?.2 (S), Q?.3 (S)
- new net SW_NODE: Q?.1 (S), Q?.2 (S), Q?.3 (S), Q?.5 (D)
- no-connect marks 0 -> 1
Other:
- moved on the sheet: U?

Commit message: Update LM5146Buck.kicad_sch
Parts:
- added C1, C2, C3, C4, C5, C7, C8, C9: 4.7u, Capacitor_SMD:C_0603_1608Metric, symbol Device:C
- added C11, C15: 68p, Capacitor_SMD:C_0603_1608Metric, symbol Device:C
- added C12: 2.2u, Capacitor_SMD:C_0603_1608Metric, symbol Device:C
- added C13: 3.9n, Capacitor_SMD:C_0603_1608Metric, symbol Device:C
- added C14: 4.7p, Capacitor_SMD:C_0603_1608Metric, symbol Device:C
- added C6: 0.1u, Capacitor_SMD:C_0603_1608Metric, symbol Device:C
- added L1: 5.6u, symbol Device:L
- added R1: 200k, Resistor_SMD:R_0603_1608Metric, symbol Device:R
- added R4: 4.87k, Resistor_SMD:R_0603_1608Metric, symbol Device:R
- added R5: 22.1k, Resistor_SMD:R_0603_1608Metric, symbol Device:R
- added R6: 845R, Resistor_SMD:R_0603_1608Metric, symbol Device:R
- added R7: 20k, Resistor_SMD:R_0603_1608Metric, symbol Device:R
- added R9: 0.768k, Resistor_SMD:R_0603_1608Metric, symbol Device:R
- C10: renamed from C1; value 100n -> 47n
- R2: renamed from R1; value 511 -> 8.25k
- R3: value R -> 8.25k
- R8: renamed from R2; value 10k2 -> 4.87k
- gave numbers to parts that had none: 3
Connections:
- net GND is gone; now on net EP: U1.12 (PGND), U1.6 (AGND)
- net EP: now also C10.2, Q2.1 (S), Q2.2 (S), Q2.3 (S), R2.1, R3.2, C1.1, C12.1, C14.1, C2.1, C3.1, C4.1, C5.1, C7.1, C8.1, C9.1, R9.1
- net SW_NODE: now also U1.19 (SW), C6.1, L1.1, R6.2
- net at R8.1: now also C13.2
- net FB: now reaches R8.2
- net FB: now also U1.5 (FB), C11.1, C15.2, R5.1, R9.2
- net SS_TRK: now reaches C10.1
- net SS_TRK: now also U1.3 (SS/TRK)
- net EN_UVLO: now reaches U1.1 (EN/UVLO)
- net EN_UVLO: now also R2.2, R1.1
- net PGOOD: now reaches U1.10 (PGOOD)
- net PGOOD: now also R7.1
- net at U1.11 (ILIM): now also C14.2, R6.1
- net Vcc: now reaches U1.14 (VCC)
- net Vcc: now also C12.2, R7.2
- net at U1.17 (BST): now also C6.2
- net RT: now reaches U1.2 (RT)
- net RT: now also R3.1
- net Vin: now reaches U1.20 (VIN)
- net Vin: now also Q1.5 (D), C1.2, C2.2, C3.2, C4.2, C5.2, R1.2
- net COMP: now reaches U1.4 (COMP)
- net COMP: now also C13.1, C15.1
- new net: C11.2, R4.1
- new net Vout: C7.2, C8.2, C9.2, L1.2, R4.2, R5.2
- no-connect marks 1 -> 3
Other:
- moved on the sheet: C10, Q1, Q2, R2, R8, U1

Commit message: Update LM5146Buck.kicad_sch
Parts:
- added C16: 1000u, Capacitor_SMD:C_0603_1608Metric, symbol Device:C
- added D1, D2, D3, D4, D5, D6: 1N5402, Diode_THT:D_DO-201AD_P15.24mm_Horizontal, symbol Diode:1N5402
- added J1, J2: Conn_01x02, Connector_AMASS:AMASS_XT60PW-M_1x02_P7.20mm_Horizontal, symbol Connector_Generic:Conn_01x02
- added J3: Conn_01x03, symbol Connector_Generic:Conn_01x03
- added RV1: 1k, symbol Device:R_Potentiometer
- R9: value 0.768k -> 511R
- U1: CREATOR (none) -> DIZAR; Check_prices (none) -> https://www.snapeda.com/parts/LM5146RGYR/Texas+Instruments/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; DUPLICATE (none) -> LM5146RGYR.A-,-LM5146RGYRG4-,-LM5146RGYRG4.A; DigiKey_Part_Number (none) -> 296-LM5146RGYRCT-ND; MANUFACTURER (none) -> Texas Instruments; MAXIMUM_PACKAGE_HEIGHT (none) -> 1.0mm; MF (none) -> Texas Instruments; MP (none) -> LM5146RGYR; PARTREV (none) -> A; Package (none) -> VFQFN-20 Texas Instruments; STANDARD (none) -> Manufacturer Recommendations; SnapEDA_Link (none) -> https://www.snapeda.com/parts/LM5146RGYR/Texas+Instruments/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
Connections:
- net EP: now also C16.1, D4.2 (A), D5.2 (A), D6.2 (A), J1.2 (Pin_2), J2.2 (Pin_2)
- net FB: now also RV1.3; no longer R9.2
- net Vin: now also C16.2, D1.1 (K), D2.1 (K), D3.1 (K), J1.1 (Pin_1)
- net Vout: now also J2.1 (Pin_1)
- new net: R9.2, RV1.1, RV1.2
- new net: D1.2 (A), D4.1 (K), J3.1 (Pin_1)
- new net: D2.2 (A), D5.1 (K), J3.2 (Pin_2)
- new net: D3.2 (A), D6.1 (K), J3.3 (Pin_3)
Other:
- note added: "12-30V"
- moved on the sheet: C1, C10, C11, C12, C13, C14, C15, C2, C3, C4, C5, C6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
