File: LM5146Buck/LM5146Buck.kicad_sch (KiCad schematic)
At the start: 39 parts, among them J1 Conn_01x02, J2 Conn_01x02, J3 Conn_01x03, U1 LM5146RGYR

Commit message: Update LM5146Buck.kicad_sch
Parts:
- Q1, Q2: value (none) -> BSC040N10NS5; footprint Package_TO_SOT_SMD:TDSON-8-1 -> 0_SuperSO:Infineon_PG-TDSON-8_6.15x5.15mm
Changed lines of the file:
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@@
 		(in_pos_files yes)
 		(dnp no)
-		(fields_autoplaced yes)
 		(property "Reference" "Q2"
 			(at 275.59 151.13 0)
@@
 			)
 		)
-		(property "Value" ""
-			(at 275.59 152.4 0)
+		(property "Value" "BSC040N10NS5"
+			(at 275.59 153.162 0)
 			(show_name no)
 			(do_not_autoplace no)
@@
 			)
 		)
-		(property "Footprint" "Package_TO_SOT_SMD:TDSON-8-1"
+		(property "Footprint" "0_SuperSO:Infineon_PG-TDSON-8_6.15x5.15mm"
 			(at 274.32 153.035 0)
 			(hide yes)
@@
 		(in_pos_files yes)
 		(dnp no)
-		(fields_autoplaced yes)
 		(property "Reference" "Q1"
-			(at 275.59 127 0)
+			(at 275.082 125.984 0)
 			(show_name no)
 			(do_not_autoplace no)
@@
 			)
 		)
-		(property "Value" ""
-			(at 275.59 128.27 0)
+		(property "Value" "BSC040N10NS5"
+			(at 274.574 128.016 0)
 			(show_name no)
 			(do_not_autoplace no)
@@
 			)
 		)
-		(property "Footprint" "Package_TO_SOT_SMD:TDSON-8-1"
+		(property "Footprint" "0_SuperSO:Infineon_PG-TDSON-8_6.15x5.15mm"
 			(at 274.32 128.905 0)
 			(hide yes)

Commit message: Update LM5146Buck.kicad_sch
Parts:
- C1, C2, C3, C4, C5, C7, C8, C9: footprint Capacitor_SMD:C_0603_1608Metric -> Capacitor_SMD:C_1210_3225Metric; LCSC (none) -> C381466
- C10, C14, C6: LCSC (none) -> C1622
- C11, C15: LCSC (none) -> C123587
- C12: LCSC (none) -> C23630
- C13: LCSC (none) -> C1618
- L1: footprint (none) -> 0_MDA1350-6R8M:MDA; LCSC (none) -> C2847572
- Q1, Q2: LCSC (none) -> C534334
- R1: LCSC (none) -> C25811
- R2, R3: LCSC (none) -> C23113
- R4, R8: LCSC (none) -> C137709
- R5: LCSC (none) -> C25961
- R6: LCSC (none) -> C227933
- R7: LCSC (none) -> C4184
- R9: LCSC (none) -> C23195
- U1: LCSC (none) -> C3188679
Other:
- note added: "MDA1350-6R8M"
